File: neptune-imu/neptune-imu.kicad_pcb (KiCad board)
At the start: 6 copper layers, 50 x 50 mm, 44 parts, among them J1 Connector, J2 Left through connector, J3 Right through connector, SW1 reset, U1 STM32L432KCUx, U2 MAX31865xTP, U3 MAX31865xTP, U4 MAX31865xTP, U5 AP2112K-3.3, U6 BME680_1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

Commit message: almost ready
Parts:
- removed C3: 100nF, Capacitor_SMD:C_0402_1005Metric
- removed D1: User LED, LED_SMD:LED_0603_1608Metric
- removed R5: 1k, Resistor_SMD:R_0402_1005Metric
- added C22: 4.7uF, Capacitor_SMD:C_0603_1608Metric, F.Cu at (91.4, 41.3)
- added TP3: 3v3, TestPoint:TestPoint_Pad_1.5x1.5mm, F.Cu at (115.6, 43.3)
- added TP4: GND, TestPoint:TestPoint_Pad_1.5x1.5mm, F.Cu at (115.6, 40.1)
- added TP5: Vbus, TestPoint:TestPoint_Pad_1.5x1.5mm, F.Cu at (115.6, 46.6)
- C1: footprint Capacitor_SMD:C_0402_1005Metric -> Capacitor_SMD:C_0603_1608Metric
- C11, C12, C5, C6, C8, C9: footprint Capacitor_SMD:C_0402_1005Metric -> Capacitor_SMD:C_0201_0603Metric
- SW1: moved to B.Cu
- TP1, TP2: footprint TestPoint:TestPoint_Pad_2.0x2.0mm -> TestPoint:TestPoint_Pad_1.0x1.0mm
- U5: footprint Package_TO_SOT_SMD:SOT-23-5 -> neptune-imu-footprints:ap2112
- moved C15 96.1 mm to (122.6, 43.7)
- moved C14 92.4 mm to (122.1, 49.5), turned to 180 degrees
- moved U5 92.1 mm to (122.6, 46.6), turned to 90 degrees
- moved C1 73.8 mm to (91.7, 39.4), turned to 180 degrees
- moved U2 69.7 mm to (91.9, 80.0)
- moved TP2 69.3 mm to (83.6, 46.1)
- moved U4 67.6 mm to (114.9, 80.0)
- moved TP1 65.1 mm to (83.6, 48.6), turned to -90 degrees
- moved R1 64.4 mm to (84.1, 44.5), turned to 180 degrees
- moved SW1 64.4 mm to (91.7, 39.4), turned to 180 degrees
- moved U3 64.1 mm to (103.4, 80.0)
- moved TH3 58.0 mm to (114.5, 85.3)
- moved R4 57.1 mm to (110.4, 79.7), turned to -90 degrees
- moved C13 56.6 mm to (114.5, 83.6)
- moved C11 56.2 mm to (114.3, 76.1), turned to -90 degrees
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Connections:
- J2 pad 2: /I2C_1_SDA -> /I2C1_SDA
- J2 pad 4: /I2C_1_SCL -> /I2C1_SCL
- U1 pad 10: unconnected-(U1-PA4-Pad10) -> /BME690_CS3
- U1 pad 14: /BME690_CS1 -> /BME690_CS2
- U1 pad 15: /BME690_CS2 -> /BME690_CS1
- U1 pad 18: /BME690_CS3 -> unconnected-(U1-PA8-Pad18)
- U1 pad 2: /MAX31865_DRDY2 -> /MAX31865_DRDY1
- U1 pad 25: Net-(D1-A) -> unconnected-(U1-PA15-Pad25)
- U1 pad 6: /MAX31865_DRDY1 -> /MAX31865_DRDY2
Routing:
- net SPI1_MISO: track 1.50 -> 115.7 mm, vias 2 -> 7
- net SPI1_SCK: track 1.63 -> 103.6 mm, vias 2 -> 7
- net SPI1_MOSI: track 1.63 -> 102.4 mm, vias 2 -> 7
- net /MAX31865_CS3: track 0.00 -> 63.0 mm, vias 0 -> 2
- net /MAX31865_DRDY3: track 0.00 -> 53.4 mm, vias 0 -> 2
- net /MAX31865_CS2: track 0.00 -> 51.4 mm, vias 0 -> 2
- net GND: track 12.7 -> 55.2 mm, vias 11 -> 78
- net /MAX31865_DRDY2: track 0.00 -> 41.1 mm, vias 0 -> 2
- net /MAX31865_CS1: track 0.00 -> 41.0 mm, vias 0 -> 2
- net /MAX31865_DRDY1: track 0.00 -> 31.3 mm, vias 0 -> 2
- net /USART1_RX: track 0.00 -> 30.3 mm, vias 0 -> 1
- net /BME690_CS3: track 0.00 -> 24.2 mm
- net /VOUT_A1: track 0.00 -> 22.9 mm
- net /reset: track 0.00 -> 22.9 mm, vias 0 -> 3
- net /USART1_TX: track 0.00 -> 22.5 mm, vias 0 -> 1
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- added copper zone on In2.Cu, net +3.3V
- added copper zone on In1.Cu, net GND
- added copper zone on In4.Cu, net GND
Other:
- board text added: "3v3"
- board text added: "Boot0"
- board text added: "GND"
- board text added: "Reset"
- board text added: "Vbus"
