File: neptune-env/bme690.kicad_sch (KiCad schematic)
At the start: 9 parts, among them U6 BME680_1, U7 BME680_2, U8 BME680_3

Commit message: project naming updated
Parts:
- U6, U7, U8: footprint neptune-imu-footprints:Bosch_LGA-8_3x3mm_P0.8mm_ClockwisePinNumbering -> neptune-env-footprints:Bosch_LGA-8_3x3mm_P0.8mm_ClockwisePinNumbering
Changed lines of the file:
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@@
 			)
 		)
-		(property "Footprint" "neptune-imu-footprints:Bosch_LGA-8_3x3mm_P0.8mm_ClockwisePinNumbering"
+		(property "Footprint" "neptune-env-footprints:Bosch_LGA-8_3x3mm_P0.8mm_ClockwisePinNumbering"
 			(at 267.97 78.74 0)
 			(effects
@@
 			)
 		)
-		(property "Footprint" "neptune-imu-footprints:Bosch_LGA-8_3x3mm_P0.8mm_ClockwisePinNumbering"
+		(property "Footprint" "neptune-env-footprints:Bosch_LGA-8_3x3mm_P0.8mm_ClockwisePinNumbering"
 			(at 95.25 78.74 0)
 			(effects
@@
 			)
 		)
-		(property "Footprint" "neptune-imu-footprints:Bosch_LGA-8_3x3mm_P0.8mm_ClockwisePinNumbering"
+		(property "Footprint" "neptune-env-footprints:Bosch_LGA-8_3x3mm_P0.8mm_ClockwisePinNumbering"
 			(at 181.61 78.74 0)
 			(effects
