File: neptune-env/rtd.kicad_sch (KiCad schematic)
At the start: 18 parts, among them U2 MAX31865xTP, U3 MAX31865xTP, U4 MAX31865xTP

Commit message: project naming updated
Parts:
- TH1, TH2, TH3: footprint neptune-imu-footprints:yageo_m1020 -> neptune-env-footprints:yageo_m1020
- U2, U3, U4: footprint neptune-imu-footprints:MAX31865 -> neptune-env-footprints:MAX31865
Changed lines of the file:
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@@
 			)
 		)
-		(property "Footprint" "neptune-imu-footprints:yageo_m1020"
+		(property "Footprint" "neptune-env-footprints:yageo_m1020"
 			(at 92.71 100.33 0)
 			(effects
@@
 			)
 		)
-		(property "Footprint" "neptune-imu-footprints:MAX31865"
+		(property "Footprint" "neptune-env-footprints:MAX31865"
 			(at 233.68 111.76 0)
 			(effects
@@
 			)
 		)
-		(property "Footprint" "neptune-imu-footprints:yageo_m1020"
+		(property "Footprint" "neptune-env-footprints:yageo_m1020"
 			(at 265.43 100.33 0)
 			(effects
@@
 			)
 		)
-		(property "Footprint" "neptune-imu-footprints:MAX31865"
+		(property "Footprint" "neptune-env-footprints:MAX31865"
 			(at 60.96 111.76 0)
 			(effects
@@
 			)
 		)
-		(property "Footprint" "neptune-imu-footprints:MAX31865"
+		(property "Footprint" "neptune-env-footprints:MAX31865"
 			(at 147.32 111.76 0)
 			(effects
@@
 			)
 		)
-		(property "Footprint" "neptune-imu-footprints:yageo_m1020"
+		(property "Footprint" "neptune-env-footprints:yageo_m1020"
 			(at 179.07 100.33 0)
 			(effects
