File: neptune-env/neptune-env.kicad_pcb (KiCad board)
At the start: 6 copper layers, 50 x 50 mm, 45 parts, among them J1 Connector, J2 Left through connector, J3 Right through connector, SW1 reset, U1 STM32L432KCUx, U2 MAX31865xTP, U3 MAX31865xTP, U4 MAX31865xTP, U5 AP2112K-3.3, U6 BME680_1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

Commit message: project naming updated
Parts:
- J1: footprint neptune-imu-footprints:HDR-SMD_8P-P2.00-H-F-W9.2 -> neptune-env-footprints:HDR-SMD_8P-P2.00-H-F-W9.2
- J2, J3: footprint neptune-imu-footprints:gaia_connector -> neptune-env-footprints:gaia_connector
- SW1: footprint neptune-imu-footprints:KEY-SMD_L4.0-W3.0-LS4.9-1 -> neptune-env-footprints:KEY-SMD_L4.0-W3.0-LS4.9-1
- TH1, TH2, TH3: footprint neptune-imu-footprints:yageo_m1020 -> neptune-env-footprints:yageo_m1020
- U1: footprint neptune-imu-footprints:STM32L432KCUx -> neptune-env-footprints:STM32L432KCUx
- U2, U3, U4: footprint neptune-imu-footprints:MAX31865 -> neptune-env-footprints:MAX31865
- U5: footprint neptune-imu-footprints:ap2112 -> neptune-env-footprints:ap2112
- U6, U7, U8: footprint neptune-imu-footprints:Bosch_LGA-8_3x3mm_P0.8mm_ClockwisePinNumbering -> neptune-env-footprints:Bosch_LGA-8_3x3mm_P0.8mm_ClockwisePinNumbering

Commit message: some advancements
Parts:
- moved TH1 0.33 mm to (91.9, 85.3)
- moved TH2 0.33 mm to (103.4, 85.3)
- moved TH3 0.33 mm to (114.9, 85.3)

Commit message: some final things to do
Parts:
- moved TP4 4.11 mm to (117.1, 43.9)
- moved TP3 3.34 mm to (117.1, 40.3)
- moved TP5 1.73 mm to (117.1, 47.4)
- moved C14 0.10 mm to (122.1, 49.6)
- moved C15 0.10 mm to (122.6, 43.8)
- moved U5 0.10 mm to (122.6, 46.7)
Routing:
- net +3.3V: track 28.1 -> 30.5 mm
- net /VOUT_A1: track 22.9 -> 21.1 mm
- net SPI1_SCK: track 103.6 -> 102.2 mm
- net SPI1_MISO: track 115.7 -> 114.4 mm
- net SPI1_MOSI: track 102.4 -> 101.3 mm
Other:
- board text added: "Environmental Measurement Unit"
- board text added: "revision 1.0 Project Neptune"
- board text removed: "Vbus"

Commit message: ready
final check needed
Parts:
- moved C9 0.47 mm to (101.9, 76.1), turned to 90 degrees
- moved C8 0.31 mm to (102.8, 76.1), turned to -90 degrees
Other:
- outline, holes or cut-outs redrawn

Commit message: working on my PC
Routing:
- net +3.3V: track 30.3 -> 31.1 mm

Commit message: ready
Connections:
- J2 pad 1: unconnected-(J2-Pin_1-Pad1) -> /I2C_2_SDA
- J2 pad 10: unconnected-(J2-Pin_10-Pad10) -> GND
- J2 pad 2: /I2C1_SDA -> unconnected-(J2-Pin_2-Pad2)
- J2 pad 3: unconnected-(J2-Pin_3-Pad3) -> /I2C_2_SCL
- J2 pad 4: /I2C1_SCL -> unconnected-(J2-Pin_4-Pad4)
- U1 pad 29: /I2C1_SCL -> /I2C_2_SCL
- U1 pad 30: /I2C1_SDA -> /I2C_2_SDA
Routing:
- net /I2C_2_SCL: track 0.00 -> 14.1 mm, vias 0 -> 1
- net /I2C1_SCL: track 11.7 -> 0.00 mm, vias 1 -> 0
- net /I2C_2_SDA: track 0.00 -> 9.19 mm, vias 0 -> 1
- net /I2C1_SDA: track 7.73 -> 0.00 mm, vias 1 -> 0
- net /VOUT_A1: track 21.1 -> 20.5 mm
- net GND: vias 78 -> 85
Other:
- board text added: "Vout"

Commit message: Review: OK for production
Other:
- board text added: "3V3"
- board text added: "B0"
- board text added: "RESET"
- board text added: "RST"
- board text added: "VIN"
- board text removed: "3v3"
- board text removed: "Boot0"
- board text removed: "Reset"
- board text removed: "Vout"
Changed lines of the file:
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@@
 		)
 	)
-	(gr_text "3v3"
+	(gr_text "3V3"
 		(at 119.046938 40.33 90)
 		(layer "F.SilkS")
@@
 		)
 	)
-	(gr_text "Vout"
+	(gr_text "VIN"
 		(at 119.046938 47.430001 90)
 		(layer "F.SilkS")
@@
 		)
 	)
-	(gr_text "Reset"
+	(gr_text "RST"
 		(at 82.2 48.641 270)
 		(layer "F.SilkS")
 		(effects
 			(font
-				(size 0.5 0.5)
-				(thickness 0.1)
+				(size 0.6 0.6)
+				(thickness 0.12)
 				(bold yes)
 			)
 		)
 	)
-	(gr_text "Boot0"
+	(gr_text "B0"
 		(at 82.2 46.086 270)
 		(layer "F.SilkS")
 		(effects
 			(font
-				(size 0.5 0.5)
-				(thickness 0.1)
+				(size 0.6 0.6)
+				(thickness 0.12)
 				(bold yes)
 			)
@@
 		)
 	)
-	(gr_text "Reset"
-		(at 91.660938 37.037 -180)
+	(gr_text "RESET"
+		(at 91.660938 37.037 180)
 		(layer "B.SilkS")
 		(effects

Commit message: fixing bugs, production
Routing:
- net GND: track 54.8 -> 37.5 mm
- net +3.3V: track 31.1 -> 30.0 mm
- net /I2C_2_SCL: track 14.1 -> 13.3 mm
- net /SWDIO: track 13.9 -> 13.2 mm
- net /SWCLK: track 17.3 -> 16.6 mm
- net /USART1_RX: track 30.3 -> 29.7 mm
