File: neptune-env/neptune-env.kicad_pcb (KiCad board)
At the start: 6 copper layers, 50 x 50 mm, 45 parts, among them J1 Connector, J2 Left through connector, J3 Right through connector, SW1 reset, U1 STM32L432KCUx, U2 MAX31865xTP, U3 MAX31865xTP, U4 MAX31865xTP, U5 AP2112K-3.3, U6 BME680_1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

Commit message: v1.1 - PRODUCTION
Header FIX
Connections:
- J2 pad 6: unconnected-(J2-Pin_6-Pad6) -> GND
- J2 pad 7: GND -> unconnected-(J2-Pin_7-Pad7)
- J2 pad 8: unconnected-(J2-Pin_8-Pad8) -> GND
Routing:
- net /BME690_CS3: track 24.2 -> 23.6 mm
Other:
- board text added: "revision 1.1 Project Neptune"
- board text removed: "revision 1.0 Project Neptune"
