File: neptune-env/neptune-env.kicad_sch (KiCad schematic)
At the start: 18 parts, among them J1 Connector, J2 Left through connector, J3 Right through connector, SW1 reset, U1 STM32L432KCUx, U5 AP2112K-3.3

Commit message: project naming updated
Parts:
- J1: footprint neptune-imu-footprints:HDR-SMD_8P-P2.00-H-F-W9.2 -> neptune-env-footprints:HDR-SMD_8P-P2.00-H-F-W9.2
- J2, J3: footprint neptune-imu-footprints:gaia_connector -> neptune-env-footprints:gaia_connector
- SW1: footprint neptune-imu-footprints:KEY-SMD_L4.0-W3.0-LS4.9-1 -> neptune-env-footprints:KEY-SMD_L4.0-W3.0-LS4.9-1
- U1: footprint neptune-imu-footprints:STM32L432KCUx -> neptune-env-footprints:STM32L432KCUx
- U5: footprint neptune-imu-footprints:ap2112 -> neptune-env-footprints:ap2112
Changed lines of the file:
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@@
 			)
 		)
-		(property "Footprint" "neptune-imu-footprints:HDR-SMD_8P-P2.00-H-F-W9.2"
+		(property "Footprint" "neptune-env-footprints:HDR-SMD_8P-P2.00-H-F-W9.2"
 			(at 143.51 48.26 0)
 			(effects
@@
 			)
 		)
-		(property "Footprint" "neptune-imu-footprints:STM32L432KCUx"
+		(property "Footprint" "neptune-env-footprints:STM32L432KCUx"
 			(at 57.15 90.17 0)
 			(effects
@@
 			)
 		)
-		(property "Footprint" "neptune-imu-footprints:KEY-SMD_L4.0-W3.0-LS4.9-1"
+		(property "Footprint" "neptune-env-footprints:KEY-SMD_L4.0-W3.0-LS4.9-1"
 			(at 43.18 26.67 0)
 			(effects
@@
 			)
 		)
-		(property "Footprint" "neptune-imu-footprints:gaia_connector"
+		(property "Footprint" "neptune-env-footprints:gaia_connector"
 			(at 237.49 80.01 0)
 			(effects
@@
 			)
 		)
-		(property "Footprint" "neptune-imu-footprints:ap2112"
+		(property "Footprint" "neptune-env-footprints:ap2112"
 			(at 157.48 74.295 0)
 			(effects
@@
 			)
 		)
-		(property "Footprint" "neptune-imu-footprints:gaia_connector"
+		(property "Footprint" "neptune-env-footprints:gaia_connector"
 			(at 237.49 44.45 0)
 			(effects
@@
 		)
 		(instances
-			(project "neptune-imu"
+			(project "neptune-env"
 				(path "/63071433-ee88-4c4a-9cea-cf45be729e9d"
 					(page "3")
@@
 		)
 		(instances
-			(project "neptune-imu"
+			(project "neptune-env"
 				(path "/63071433-ee88-4c4a-9cea-cf45be729e9d"
 					(page "2")

Commit message: some final things to do
Other:
- moved on the sheet: J2, J3

Commit message: ready
Connections:
- net GND: now also J2.10 (Pin_10)
- net I2C_2_SDA: now reaches J2.1 (Pin_1)
- net I2C_2_SDA: now also U1.30 (PB7)
- net I2C_2_SCL: now reaches J2.3 (Pin_3)
- net I2C_2_SCL: now also U1.29 (PB6)
- net I2C1_SCL: no longer names the net of J2.4 (Pin_4)
- net I2C1_SCL: no longer U1.29 (PB6)
- net I2C1_SDA: no longer names the net of J2.2 (Pin_2)
- net I2C1_SDA: no longer U1.30 (PB7)
- no-connect marks 31 -> 30
Changed lines of the file:
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@@
-	)
-	(no_connect
-		(at 210.82 27.94)
 	)
 	(no_connect
@@
 	)
 	(no_connect
-		(at 210.82 30.48)
-	)
-	(no_connect
 		(at 210.82 40.64)
 	)
@@
 	)
 	(no_connect
+		(at 223.52 27.94)
+	)
+	(no_connect
 		(at 223.52 33.02)
 	)
@@
 	)
 	(no_connect
-		(at 223.52 38.1)
-	)
-	(no_connect
 		(at 54.61 72.39)
 	)
@@
 	)
 	(no_connect
+		(at 223.52 30.48)
+	)
+	(no_connect
 		(at 251.46 40.64)
 	)
@@
 	(wire
 		(pts
-			(xy 223.52 30.48) (xy 224.79 30.48)
-		)
-		(stroke
-			(width 0)
-			(type default)
-		)
-	)
-	(wire
-		(pts
 			(xy 91.44 118.11) (xy 92.71 118.11)
 		)
@@
 	(wire
 		(pts
+			(xy 209.55 27.94) (xy 210.82 27.94)
+		)
+		(stroke
+			(width 0)
+			(type default)
+		)
+	)
+	(wire
+		(pts
 			(xy 36.83 41.91) (xy 40.64 41.91)
 		)
@@
 	(wire
 		(pts
-			(xy 223.52 27.94) (xy 224.79 27.94)
-		)
-		(stroke
-			(width 0)
-			(type default)
-		)
-	)
-	(wire
-		(pts
 			(xy 45.72 118.11) (xy 46.99 118.11)
 		)
@@
 	(wire
 		(pts
+			(xy 223.52 38.1) (xy 226.06 38.1)
+		)
+		(stroke
+			(width 0)
+			(type default)
+		)
+	)
+	(wire
+		(pts
 			(xy 53.34 77.47) (xy 54.61 77.47)
 		)
@@
 		(pts
 			(xy 80.01 46.99) (xy 81.28 46.99)
+		)
+		(stroke
+			(width 0)
+			(type default)
+		)
+	)
+	(wire
+		(pts
+			(xy 209.55 30.48) (xy 210.82 30.48)
 		)
 		(stroke
@@
 		)
 	)
-	(label "I2C1_SDA"
+	(label "I2C_2_SDA"
 		(at 53.34 80.01 180)
 		(effects
@@
 		)
 	)
+	(label "I2C_2_SDA"
+		(at 209.55 27.94 180)
+		(effects
+			(font
+				(size 1.27 1.27)
+			)
+			(justify right bottom)
+		)
+	)
 	(label "VOUT_A1"
 		(at 264.16 27.94 0)
@@
 		)
 	)
+	(label "I2C_2_SCL"
+		(at 209.55 30.48 180)
+		(effects
+			(font
+				(size 1.27 1.27)
+			)
+			(justify right bottom)
+		)
+	)
 	(label "MAX31865_DRDY3"
 		(at 53.34 59.69 180)
@@
 		)
 	)
-	(label "I2C1_SDA"
-		(at 224.79 27.94 0)
-		(effects
-			(font
-				(size 1.27 1.27)
-			)
-			(justify left bottom)
-		)
-	)
-	(label "I2C1_SCL"
-		(at 224.79 30.48 0)
-		(effects
-			(font
-				(size 1.27 1.27)
-			)
-			(justify left bottom)
-		)
-	)
 	(label "reset"
 		(at 52.07 39.37 90)
@@
 		)
 	)
-	(label "I2C1_SCL"
+	(label "I2C_2_SCL"
 		(at 53.34 77.47 180)
 		(effects
@@
 					(unit 1)
 				)
+			)
+		)
+	)
+	(symbol
+		(lib_id "power:GND")
+		(at 226.06 38.1 90)
+		(unit 1)
+		(exclude_from_sim no)
+		(in_bom yes)
+		(on_board yes)
+		(dnp no)
+		(fields_autoplaced yes)
+		(property "Reference" "#PWR059"
+			(at 232.41 38.1 0)
+			(effects
+				(font
+					(size 1.27 1.27)
+				)
+				(hide yes)
+			)
+		)
+		(property "Value" "GND"
+			(at 229.87 38.0999 90)
+			(effects
+				(font
+					(size 1.27 1.27)
+				)
+				(justify right)
+			)
+		)
+		(property "Footprint" ""
+			(at 226.06 38.1 0)
+			(effects
+				(font
+					(size 1.27 1.27)
+				)
+				(hide yes)
+			)
+		)
+		(property "Datasheet" ""
+			(at 226.06 38.1 0)
+			(effects
+				(font
+					(size 1.27 1.27)
+				)
+				(hide yes)
+			)
+		)
+		(property "Description" "Power symbol creates a global label with name \"GND\" , ground"
+			(at 226.06 38.1 0)
+			(effects
+				(font
+					(size 1.27 1.27)
+				)
+				(hide yes)
+			)
+		)
+		(pin "1"
+		)
+		(instances
+			(project "neptune-env"
+				(path "/63071433-ee88-4c4a-9cea-cf45be729e9d"
+					(reference "#PWR059")
+					(unit 1)
+				)

Commit message: v1.1 - PRODUCTION
Header FIX
Connections:
- net GND: now also J2.6 (Pin_6), J2.8 (Pin_8); no longer J2.7 (Pin_7)
- no-connect marks 30 -> 29
Changed lines of the file:
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@@
 	)
 	(no_connect
-		(at 223.52 33.02)
-	)
-	(no_connect
-		(at 223.52 35.56)
-	)
-	(no_connect
 		(at 80.01 74.93)
 	)
@@
 	)
 	(no_connect
+		(at 210.82 35.56)
+	)
+	(no_connect
 		(at 210.82 45.72)
 	)
@@
 	(wire
 		(pts
-			(xy 208.28 35.56) (xy 210.82 35.56)
-		)
-		(stroke
-			(width 0)
-			(type default)
-		)
-	)
-	(wire
-		(pts
 			(xy 76.2 27.94) (xy 76.2 30.48)
 		)
@@
 	)
 	(symbol
-		(lib_id "power:GND")
-		(at 208.28 35.56 270)
-		(unit 1)
-		(exclude_from_sim no)
-		(in_bom yes)
-		(on_board yes)
-		(dnp no)
-		(fields_autoplaced yes)
-		(property "Reference" "#PWR075"
-			(at 201.93 35.56 0)
-			(effects
-				(font
-					(size 1.27 1.27)
-				)
-				(hide yes)
-			)
-		)
-		(property "Value" "GND"
-			(at 204.47 35.5599 90)
-			(effects
-				(font
-					(size 1.27 1.27)
-				)
-				(justify right)
-			)
-		)
-		(property "Footprint" ""
-			(at 208.28 35.56 0)
-			(effects
-				(font
-					(size 1.27 1.27)
-				)
-				(hide yes)
-			)
-		)
-		(property "Datasheet" ""
-			(at 208.28 35.56 0)
-			(effects
-				(font
-					(size 1.27 1.27)
-				)
-				(hide yes)
-			)
-		)
-		(property "Description" "Power symbol creates a global label with name \"GND\" , ground"
-			(at 208.28 35.56 0)
-			(effects
-				(font
-					(size 1.27 1.27)
-				)
-				(hide yes)
-			)
-		)
-		(pin "1"
-		)
-		(instances
-			(project "neptune-imu"
-				(path "/63071433-ee88-4c4a-9cea-cf45be729e9d"
-					(reference "#PWR075")
-					(unit 1)
-				)
-			)
-		)
-	)
-	(symbol
 		(lib_id "power:+3.3V")
 		(at 160.02 40.64 180)
@@
 	)
 	(symbol
+		(lib_id "power:GND")
+		(at 223.52 33.02 90)
+		(unit 1)
+		(exclude_from_sim no)
+		(in_bom yes)
+		(on_board yes)
+		(dnp no)
+		(fields_autoplaced yes)
+		(property "Reference" "#PWR061"
+			(at 229.87 33.02 0)
+			(effects
+				(font
+					(size 1.27 1.27)
+				)
+				(hide yes)
+			)
+		)
+		(property "Value" "GND"
+			(at 227.33 33.0199 90)
+			(effects
+				(font
+					(size 1.27 1.27)
+				)
+				(justify right)
+			)
+		)
+		(property "Footprint" ""
+			(at 223.52 33.02 0)
+			(effects
+				(font
+					(size 1.27 1.27)
+				)
+				(hide yes)
+			)
+		)
+		(property "Datasheet" ""
+			(at 223.52 33.02 0)
+			(effects
+				(font
+					(size 1.27 1.27)
+				)
+				(hide yes)
+			)
+		)
+		(property "Description" "Power symbol creates a global label with name \"GND\" , ground"
+			(at 223.52 33.02 0)
+			(effects
+				(font
+					(size 1.27 1.27)
+				)
+				(hide yes)
+			)
+		)
+		(pin "1"
+		)
+		(instances
+			(project "neptune-env"
+				(path "/63071433-ee88-4c4a-9cea-cf45be729e9d"
+					(reference "#PWR061")
+					(unit 1)
+				)
+			)
+		)
+	)
+	(symbol
 		(lib_id "Connector_Generic:Conn_02x10_Odd_Even")
 		(at 215.9 38.1 0)
@@
 					(unit 1)
 				)
+			)
+		)
+	)
+	(symbol
+		(lib_id "power:GND")
+		(at 223.52 35.56 90)
+		(unit 1)
+		(exclude_from_sim no)
+		(in_bom yes)
+		(on_board yes)
+		(dnp no)
+		(fields_autoplaced yes)
+		(property "Reference" "#PWR060"
+			(at 229.87 35.56 0)
+			(effects
+				(font
+					(size 1.27 1.27)
+				)
+				(hide yes)
+			)
+		)
+		(property "Value" "GND"
+			(at 227.33 35.5599 90)
+			(effects
+				(font
+					(size 1.27 1.27)
+				)
+				(justify right)
+			)
+		)
+		(property "Footprint" ""
+			(at 223.52 35.56 0)
+			(effects
+				(font
+					(size 1.27 1.27)
+				)
+				(hide yes)
+			)
+		)
+		(property "Datasheet" ""
+			(at 223.52 35.56 0)
+			(effects
+				(font
+					(size 1.27 1.27)
+				)
+				(hide yes)
+			)
+		)
+		(property "Description" "Power symbol creates a global label with name \"GND\" , ground"
+			(at 223.52 35.56 0)
+			(effects
+				(font
+					(size 1.27 1.27)
+				)
+				(hide yes)
+			)
+		)
+		(pin "1"
+		)
+		(instances
+			(project "neptune-env"
+				(path "/63071433-ee88-4c4a-9cea-cf45be729e9d"
+					(reference "#PWR060")
+					(unit 1)
+				)
